File: eagle/ports/Board1.brd (EAGLE design)
At the start: 101.6 x 54 mm, 18 parts

Commit message: WIP
Parts:
- moved JP9 1.37 mm to (15.9, 13.5)
- moved JP8 0.77 mm to (32.6, 12.6)
Connections:
- removed net RX3_D15: COMMUNICATION.7, JP8.4
- removed net RX4_D14: COMMUNICATION.8, JP8.3
- removed net SCL_D21: COMMUNICATION.1, JP8.10
- new net N$1: COMMUNICATION.2, JP8.10
- net +3V3: no longer JP12.10
- net +5V: no longer JP12.9
- net DIG52: now also JP7.1; no longer JP7.2
- net DIG53: now also JP7.2; no longer JP7.1
- net GND: now also JP12.10, JP12.9
- net PWM10: now also PWM(H).4; no longer PWM(H).3
- net PWM11: now also PWM(H).3; no longer PWM(H).4
- net PWM12: now also JP8.4
- net PWM13: now also JP8.3
- net SDA_D20: now also COMMUNICATION.1; no longer COMMUNICATION.2
Routing:
- net PWM12: track 0.00 -> 51.0 mm
- net PWM13: track 0.00 -> 48.7 mm
- net PWM11: track 0.00 -> 43.1 mm
- net PWM10: track 0.00 -> 40.2 mm
- net SDA_D20: track 0.00 -> 18.7 mm
- net TX1_D18: track 0.00 -> 18.5 mm
- net GND: track 21.8 -> 38.1 mm
- net TX2_D16: track 0.00 -> 16.0 mm
- net N$1: track 0.00 -> 12.7 mm
- net RX1_D19: track 0.63 -> 13.2 mm
- net DIG53: track 80.3 -> 92.7 mm
- net RX2_D17: track 0.00 -> 10.9 mm
- net +5V: track 10.1 -> 0.00 mm
- net DIG52: track 87.2 -> 94.2 mm
- net +3V3: track 3.43 -> 0.00 mm
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