File: eagle/ports/Board1.sch (EAGLE design)
At the start: 18 parts

Commit message: WIP
Parts:
- JP10, JP11, JP12, JP7, JP8, JP9: device pinhead:PINHD-2X5 -> pinhead+:PINHD-2X5SMT
Connections:
- removed net PWM00: JP7.1
- removed net PWM01: JP7.2
- removed net RX3_D15: COMMUNICATION.7, JP8.4
- removed net RX4_D14: COMMUNICATION.8, JP8.3
- removed net SCL_D21: COMMUNICATION.1, JP8.10
- new net N$1: COMMUNICATION.2, JP8.10
- net +3V3: no longer JP12.10
- net +5V: no longer JP12.9
- net DIG52: now also JP7.1
- net DIG53: now also JP7.2
- net GND: now also JP12.10, JP12.9
- net PWM10: now also PWM(H).4; no longer PWM(H).3
- net PWM11: now also PWM(H).3; no longer PWM(H).4
- net PWM12: now also JP8.4
- net PWM13: now also JP8.3
- net SDA_D20: now also COMMUNICATION.1; no longer COMMUNICATION.2
