File: eagle/portLights/Board2.brd (EAGLE design)
At the start: 99.1 x 55.2 mm, 68 parts

Commit message: Redesign portLights board
Parts:
- added U$1: PINHD-2X2-SMD, fab:2X02SMD
- moved R19 32.3 mm to (2.61, 4.87), turned to 90 degrees
- moved R17 28.6 mm to (11.9, 3.07), turned to 90 degrees
- moved R29 28.6 mm to (27.6, 32.1)
- moved R22 25.3 mm to (25.3, 20.7)
- moved R26 23.9 mm to (27.2, 27.0)
- moved R21 13.4 mm to (43.7, 19.8)
- moved R25 12.4 mm to (44.1, 26.5)
- moved R27 9.60 mm to (53.4, 28.7)
- moved R23 5.78 mm to (50.5, 23.4)
- moved R24 3.37 mm to (35.4, 23.6)
- moved R30 3.21 mm to (46.6, 32.8)
- moved JP8 2.26 mm to (26.2, 14.2)
- moved R28 2.14 mm to (36.1, 30.4)
- moved JP9 1.34 mm to (63.0, 27.0)
- moved JP12 1.12 mm to (73.5, 17.9)
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Connections:
- removed net N$30: JP1.8, R29.2
- new net N$18: JP9.2, R22.1
- net D21: now also COMMUNICATION.1
- net DIG22: now also JP1.16, R17.1; no longer JP9.1, R21.1
- net DIG23: now also JP1.15, R19.1; no longer JP9.2, R22.1
- net DIG24: now also JP1.14, R21.2; no longer JP9.3, R23.1
- net DIG25: now also JP1.13, R22.2; no longer JP9.4, R24.1
- net DIG26: now also JP1.12, R23.2; no longer JP9.5, R25.1
- net DIG27: now also JP1.11, R24.2; no longer JP9.6, R26.1
- net DIG28: now also JP1.10, R25.2; no longer JP9.7, R27.1
- net DIG29: now also JP1.9, R26.2; no longer JP9.8, R28.1
- net DIG30: now also JP1.8, R27.2; no longer JP9.9, R29.1
- net DIG31: now also JP1.7, R28.2; no longer JP9.10, R30.1
- net DIG32: now also R29.2; no longer R31.1
- net DIG33: now also R30.2; no longer R32.1
- net DIG34: now also R31.1; no longer R33.1
- net DIG35: now also R32.1; no longer R34.1
- net DIG36: now also R33.1; no longer R35.1
- net DIG37: now also R34.1; no longer R36.1
- net DIG38: now also R35.1; no longer R37.2
- net DIG39: now also R36.1; no longer R38.2
- net DIG40: now also R37.2; no longer R39.2
- net DIG41: now also R38.2; no longer R40.2
- net DIG42: now also R39.2; no longer R41.1
- net DIG43: now also R40.2; no longer R42.1
- net DIG44: now also R41.1; no longer R43.1
- net DIG45: now also R42.1; no longer R44.1
- net DIG46: now also R43.1; no longer R45.1
- net DIG47: now also R44.1; no longer R46.1
- net DIG48: now also R45.1; no longer R47.1
- net DIG49: now also R46.1; no longer R48.1
- net DIG50: now also R47.1; no longer R49.1
- net DIG51: now also R48.1; no longer R50.1
- net DIG52: now also R49.1; no longer R17.1
- net DIG53: now also R50.1; no longer R19.1
- net N$21: now also JP9.4, R24.1; no longer JP1.7, R30.2
- net N$22: now also JP9.6, R26.1; no longer JP1.9, R28.2
- net N$23: now also JP9.8, R28.1; no longer JP1.11, R26.2
- net N$24: now also JP9.10, R30.1; no longer JP1.13, R24.2
- net N$25: now also JP9.1, R21.1; no longer JP1.15, R22.2
- net N$26: now also JP9.3, R23.1; no longer JP1.16, R21.2
- net N$27: now also JP9.5, R25.1; no longer JP1.14, R23.2
- net N$28: now also JP9.7, R27.1; no longer JP1.12, R25.2
- net N$29: now also JP9.9, R29.1; no longer JP1.10, R27.2
- net RX3_D15: now also U$1.3
- net TX3_D14: now also U$1.4
Routing:
- net DIG53: track 0.00 -> 82.8 mm
- net DIG32: track 105.8 -> 26.3 mm
- net DIG52: track 0.00 -> 79.3 mm
- net DIG33: track 107.1 -> 49.0 mm
- net DIG30: track 0.00 -> 51.4 mm
- net DIG26: track 0.00 -> 49.9 mm
- net DIG28: track 0.00 -> 41.9 mm
- net DIG24: track 0.00 -> 40.8 mm
- net N$29: track 0.00 -> 38.1 mm
- net DIG31: track 0.00 -> 37.5 mm
- net DIG27: track 0.00 -> 35.5 mm
- net N$18: track 0.00 -> 33.9 mm
- net N$22: track 0.00 -> 32.4 mm
- net DIG29: track 0.00 -> 28.3 mm
- net DIG25: track 0.00 -> 25.3 mm
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